File: hardware/frontend/frontend.sch (KiCad schematic (older format))
At the start: 27 parts, among them P1 CONN_IO, P2 CONN_02X10, P3 CONN_01X04, SW1 PUSHB, U1 74LS74, U10 74LS173, U11 74LS32, U12 28C16, U13 28C16, U14 28C16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

Commit message: Supply ~RST to USB interface
Connections:
- net ~RST: now also P1.19 (~RST)
- no-connect marks 14 -> 13
Changed lines of the file:
@@
 Wire Wire Line
 	12800 6500 12800 6700
-NoConn ~ 13550 6600
 Wire Wire Line
 	14300 9950 14450 9950
@@
 Wire Bus Line
 	14800 5350 14800 6300
+Text GLabel 12650 6700 3    60   Input ~ 0
+~RST
+Wire Wire Line
+	12650 6700 12650 6600
+Wire Wire Line
+	12650 6600 13550 6600
 $EndSCHEMATC

Commit message: Frontend--WIP
Connections:
- net ~RERAM: now also P2.16 (P16)
- no-connect marks 13 -> 12
Changed lines of the file:
@@
 $EndComp
 NoConn ~ 14300 9650
-NoConn ~ 14300 9750
 Wire Bus Line
 	14750 8050 14750 9450
@@
 Wire Wire Line
 	12650 6600 13550 6600
+Text GLabel 14750 10150 3    60   Input ~ 0
+~RERAM
+Wire Wire Line
+	14750 10150 14750 9750
+Wire Wire Line
+	14750 9750 14300 9750
 $EndSCHEMATC
